File: pcb/MikroeAdapter/MikroeAdapter.kicad_pcb (KiCad board)
At the start: 2 copper layers, 32.8 x 86.9 mm, 19 parts, among them CON1 MIKROBUS_HOST_CONN, J1 Screw_Terminal_01x02, J2 Conn_01x03, J3 Conn_01x02, J4 Screw_Terminal_01x12, J5 Screw_Terminal_01x02, U1 ATtiny1604-SS, U2 HT75xx-1-SOT89, U3 THVD1450D

Commit message: Switched to buck converter for power so that we can run effectively off 12V
Parts:
- removed the U2 at (79.6, 58.8)
- added C1: 22u, Capacitor_SMD:C_1210_3225Metric, F.Cu at (68.3, 63.0)
- added C10: 22u, Capacitor_SMD:C_1210_3225Metric, F.Cu at (58.7, 63.8)
- added C4: 6.8nF, Capacitor_SMD:C_0603_1608Metric, F.Cu at (68.2, 69.7)
- added C5: 10p, Capacitor_SMD:C_0402_1005Metric, F.Cu at (70.0, 69.1)
- added C7: 1n, Capacitor_SMD:C_0402_1005Metric, F.Cu at (69.3, 66.1)
- added C8: 0.1u, Capacitor_SMD:C_0402_1005Metric, F.Cu at (67.1, 65.1)
- added D2: D_Schottky, Diode_SMD:D_SMA, F.Cu at (79.4, 54.1)
- added L1: 4.7uH, FNR4030:IND-SMD_L4.0-W4.0_FNR40XXS, F.Cu at (63.6, 63.4)
- added R1: 40.2k, Resistor_SMD:R_0402_1005Metric, F.Cu at (70.9, 69.1)
- added R2: 7.68k, Resistor_SMD:R_0402_1005Metric, F.Cu at (70.9, 67.2)
- added R3: 10k, Resistor_SMD:R_0402_1005Metric, F.Cu at (69.4, 67.6)
- added R4: 20, Resistor_SMD:R_0402_1005Metric, F.Cu at (65.2, 69.1)
- added R5: 604k, Resistor_SMD:R_0402_1005Metric, F.Cu at (66.8, 69.2)
- added U1: MP2331HGTL-Z, Package_TO_SOT_SMD:SOT-583-8, F.Cu at (67.1, 66.9)
- C2: value 10u -> 22u; footprint Capacitor_SMD:C_0805_2012Metric -> Capacitor_SMD:C_1210_3225Metric
- C3: value 10u -> 1u; footprint Capacitor_SMD:C_0805_2012Metric -> Capacitor_SMD:C_0603_1608Metric
- C9: renamed from C4; footprint Capacitor_SMD:C_0805_2012Metric -> Capacitor_SMD:C_0402_1005Metric
- D1: value D -> TVS; footprint Diode_SMD:D_SOD-123F -> Diode_SMD:D_SMB
- moved C2 20.8 mm to (58.7, 60.5)
- moved C3 14.9 mm to (65.0, 67.1), turned to 90 degrees
- moved D1 8.35 mm to (79.4, 61.4), turned to -90 degrees
- renumbered C1 to C6, D2 to D3, J2 to J1, J1 to J2, R1 to R6, R2 to R7, R3 to R8, R4 to R9, U1 to U2
Connections:
- C2 pad 1: Net-(D1-K) -> VCC
- C3 pad 1: VCC -> Net-(C3-Pad1)
- C3 pad 2: GND -> Net-(U1-SW)
- D1 pad 1: Net-(D1-K) -> /V_IN
- D1 pad 2: /V_IN -> GND
- J2 pad 2: /V_IN -> Net-(D2-A)
Routing:
- net /V_IN: track 9.97 -> 30.7 mm, vias 0 -> 2
- net Net-(D2-A): track 0.00 -> 12.0 mm
- net Net-(D1-K): track 8.13 -> 0.00 mm
- net Net-(U1-SW): track 0.00 -> 5.47 mm
- net /UPDI: track 67.6 -> 72.6 mm
- net GND: track 25.0 -> 28.8 mm, vias 7 -> 12
- net VCC: track 113.2 -> 110.1 mm
- net Net-(C5-Pad2): track 0.00 -> 2.85 mm
- net Net-(U1-BST): track 0.00 -> 1.71 mm
- net Net-(U1-SS): track 0.00 -> 1.66 mm
- net Net-(C3-Pad1): track 0.00 -> 1.35 mm
- net Net-(U1-EN): track 0.00 -> 1.09 mm
- net Net-(U1-FB): track 0.00 -> 1.07 mm
- net Net-(U1-PG): track 0.00 -> 1.01 mm
