File: pcb/MikroeAdapter/MikroeAdapter.kicad_sch (KiCad schematic)
At the start: 32 parts, among them CON1 MIKROBUS_HOST_CONN, J1 Conn_01x03, J2 Screw_Terminal_01x02, J3 Conn_01x02, J4 Screw_Terminal_01x12, J5 Screw_Terminal_01x02, U1 MP2331HGTL-Z, U2 ATtiny1604-SS, U3 THVD1450D

Commit message: mbq: embed the status pair in the slot; make MBQ_CMD_REGS load-bearing
The previous commit introduced two declarations that nothing used, in a
change whose purpose was removing dead code:

  - mbq_slot_status_t declared the [status | response8] wire pair, while
    mbq_slot_t separately repeated both fields. Two definitions of one
    layout, free to drift.
  - MBQ_CMD_REGS documented that a submit's length is in REGISTERS — the
    units confusion behind the two-slot bug — while modbus.c went on
    deriving first_slot and n_slots from a literal 2.

Fix both by use rather than deletion. mbq_slot_t now embeds
mbq_slot_status_t as `st`, so the in-memory and wire layouts cannot
disagree, and submit_window() derives its slot arithmetic (and its
boundary/length validation) from MBQ_CMD_REGS.

Ordering is unchanged: mbq_complete still writes st.response8 before
st.status under the same fence the status read uses. sizeof(mbq_slot_t)
== 8 still asserts. Flash is identical at 10078 B.

Verified on hardware: 400-pair soak, 14.76 pairs/s, VERDICT clean —
400 query-correct, 0 stale, 0 wrong, 0 lost, 0 out-of-order.

Co-Authored-By: Claude Opus 5 (1M context) <noreply@anthropic.com>
Claude-Session: https://claude.ai/code/session_01STSZT2DguJ8ntaDTJXvk1d
Parts:
- C6: footprint Capacitor_SMD:C_0805_2012Metric -> Capacitor_SMD:C_0402_1005Metric
Connections:
- net SW: now reaches C3.2, L1.1, U1.3 (SW)
- net PG: now reaches C7.1, U1.1 (PG)
Changed lines of the file:
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@@
+		)
+	)
+	(label "PG"
+		(at 107.95 31.75 0)
+		(effects
+			(font
+				(size 1.27 1.27)
+			)
+			(justify left bottom)
 		)
 	)
@@
 			)
 			(justify right bottom)
+		)
+	)
+	(label "SW"
+		(at 118.11 46.99 0)
+		(effects
+			(font
+				(size 1.27 1.27)
+			)
+			(justify left bottom)
 		)
 	)
@@
 			)
 		)
-		(property "Footprint" "Capacitor_SMD:C_0805_2012Metric"
+		(property "Footprint" "Capacitor_SMD:C_0402_1005Metric"
 			(at 38.1 20.6248 0)
 			(hide yes)
